File: Hardware/MainLogger.brd (EAGLE design)
At the start: 98.9 x 72.1 mm, 254 parts, among them J3 GEMS_POWER_PLUGINPUT_RT, J4 U.FL, J5 SIM_CDNANO_SF72, P1:C1 0.1uF, P1:C2 2.2uF, P1:C3 1uF, P1:C4 100uF, P1:C5 0.1uF, P1:J1 CONN_TALON_LOGGER, P1:R1 100k, P1:R2 1k, P1:R3 1k, P1:U1 SN74AUP1G08DCK, P1:U2 FXMAR2102UMLP, P1:U3 FSA2258, P1:U4 AP2411, P2:C1 0.1uF, P2:C2 2.2uF, P2:C3 1uF, P2:C4 100uF, P2:C5 0.1uF, P2:J1 CONN_TALON_LOGGER, P2:R1 100k, P2:R2 1k, P2:R3 1k, P2:U1 SN74AUP1G08DCK, P2:U2 FXMAR2102UMLP, P2:U3 FSA2258, P2:U4 AP2411, P3:C1 0.1uF, P3:C2 2.2uF, P3:C3 1uF, P3:C4 100uF, P3:C5 0.1uF, P3:J1 CONN_TALON_LOGGER, P3:R1 100k, P3:R2 1k, P3:R3 1k, P3:U1 SN74AUP1G08DCK, P3:U2 FXMAR2102UMLP, P3:U3 FSA2258, P3:U4 AP2411, P4:C1 0.1uF, P4:C2 2.2uF, P4:C3 1uF, P4:C4 100uF, P4:C5 0.1uF, P4:J1 CONN_TALON_LOGGER, P4:R1 100k, P4:R2 1k, P4:R3 1k, P4:U1 SN74AUP1G08DCK, P4:U2 FXMAR2102UMLP, P4:U3 FSA2258, P4:U4 AP2411, Q1 DMG3404, Q2 MOSFET_PCH-DMP3036SFG, Q3 MOSFET_PCH-DMP3036SFG, Q4 DMG3404, Q5 NX2301P, Q6 NX2301P, U1 FXMAR2102UMLP, U10 SN74AUP3G34DCU, U11 SIP32431TDFN, U12 LTC4412S6, U13 TCR2LE31ESV, U14 LP59073.3VYKE, U15 MIC22602, U16 BQ25616, U17 TPS61282D, U18 MCP23018QFN, U19 MCP23018QFN, U2 VEML3328, U20 MAX-M8W, U21 MCP79412SOIC, U22 HALL_EFFECT_SI7201, U23 PCA9634QFN, U24 SN74LVC1G17DCK, U25 TPL5010DDC, U26 TPL5010DDC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

Commit message: Updated v1.4 for production
Parts:
- removed P1:R1, P2:R1, P3:R1, P4:R1: 100k, bschulz_passives:R0402
- added C44, C45: 0.1uF, bschulz_passives:C0402
- added C53, C54: 1uF, bschulz_passives:C0603
- added R68: 5.6k, bschulz_passives:R0402
- added U30: TCK111G, bschulz:WCSP_6
- added U31: FPF2195BUCX, bschulz:WCSP_6
- added U32: (no value), bschulz:DCK_R-PDSO-G5
- C34: value 10uF -> 22uF
- R27: value 470R -> 220R
- R3: value 0R -> 13.3k
- R34, R36: value 10m -> 2m
- R37: value 10k -> 2.7k
- R38, R39, R43, R44: device bschulz_passives:R0603 -> bschulz_passives:R0402
- R4: value 0R -> 2k
- R50, R51, R52: value 4.7k -> 5.6k; device bschulz_passives:R0603 -> bschulz_passives:R0402
- R56: value 100k -> 130k
- R58: value 10k -> 11k
- R6, R7: value 2m -> 10m
- U11: value SIP32431TDFN -> TCK111G; device bschulz:TDFN_4 -> bschulz:WCSP_6
- moved R7 7.66 mm to (30.5, 37.8), turned to 0 degrees
- moved R14 4.10 mm to (75.7, 3.30)
- moved D6 2.67 mm to (39.9, 43.7)
- moved R24 2.03 mm to (26.7, 42.3)
- moved R40 1.67 mm to (34.7, 34.4)
- moved R2 1.65 mm to (43.8, 44.2)
- moved R1 1.65 mm to (42.7, 44.2)
- moved R15 1.65 mm to (42.7, 47.2)
- moved R27 1.52 mm to (25.5, 42.3)
- moved R26 1.02 mm to (24.4, 42.3)
- moved C11 0.99 mm to (77.3, 3.30)
- moved U11 0.77 mm to (79.2, 3.81)
- moved R52 0.63 mm to (41.9, 63.5)
- moved R28 0.51 mm to (23.2, 42.3)
- moved R50 0.38 mm to (45.0, 63.5)
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Connections:
- removed net 3V3_BULK: P1:C1.1, P1:C2.1, P1:R1.2, P1:U1.5, P1:U4.2, P1:U4.3, P2:C1.1, P2:C2.1, P2:R1.2, P2:U1.5, P2:U4.2, P2:U4.3, P3:C1.1, P3:C2.1, P3:R1.2, P3:U1.5, P3:U4.2, P3:U4.3, P4:C1.1, P4:C2.1, P4:R1.2, P4:U1.5, P4:U4.2, P4:U4.3, R7.1, U6.9
- new net 3V3_TALON: P1:C1.1, P1:C2.1, P1:U1.5, P1:U2.1, P1:U3.10, P1:U4.2, P1:U4.3, P2:C1.1, P2:C2.1, P2:U1.5, P2:U2.1, P2:U3.10, P2:U4.2, P2:U4.3, P3:C1.1, P3:C2.1, P3:U1.5, P3:U2.1, P3:U3.10, P3:U4.2, P3:U4.3, P4:C1.1, P4:C2.1, P4:U1.5, P4:U2.1, P4:U3.10, P4:U4.2, P4:U4.3, R7.2, U6.9
- new net 3V3_TALON+: C45.1, C54.1, R7.1, U30.A1, U30.B1, U31.B1, U6.10
- new net N$19: R68.2, U31.C1
- new net N$28: U31.A2, U32.4
- net !TALON1_FAULT: no longer P1:R1.1
- net !TALON2_FAULT: no longer P2:R1.1
- net !TALON3_FAULT: no longer P3:R1.1
- net !TALON4_FAULT: no longer P4:R1.1
- net 3V3_AUX: now also U11.A2, U11.B2; no longer U11.3
- net 3V3_AUX_EN: now also U30.C2, U32.2
- net 3V3_BULK+: now also C53.1, U30.A2, U30.B2; no longer R7.2, U6.10
- net 3V3_CORE: now also C44.1, U31.B2, U32.5
- net 3V3_SD: now also U11.A1, U11.B1; no longer U11.1
- net 3V3_SD_EN: now also U11.C2; no longer U11.4
- net GND: now also C44.2, C45.2, C53.2, C54.2, R68.1, U11.C1, U30.C1, U31.C2, U32.3; no longer U11.2, U11.EP
- net P1:3V3_TALON: no longer P1:U2.1, P1:U3.10
- net P1:N$1: now also P1:R2.1, P1:U3.1; no longer P1:R3.1, P1:U3.4
- net P1:N$2: now also P1:R3.1, P1:U3.3; no longer P1:R2.1, P1:U3.2
- net P2:3V3_TALON: no longer P2:U2.1, P2:U3.10
- net P2:N$1: now also P2:R2.1, P2:U3.1; no longer P2:R3.1, P2:U3.4
- net P2:N$2: now also P2:R3.1, P2:U3.3; no longer P2:R2.1, P2:U3.2
- net P3:3V3_TALON: no longer P3:U2.1, P3:U3.10
- net P3:N$1: now also P3:R2.1, P3:U3.1; no longer P3:R3.1, P3:U3.4
- net P3:N$2: now also P3:R3.1, P3:U3.3; no longer P3:R2.1, P3:U3.2
- net P4:3V3_TALON: no longer P4:U2.1, P4:U3.10
- net P4:N$1: now also P4:R2.1, P4:U3.1; no longer P4:R3.1, P4:U3.4
- net P4:N$2: now also P4:R3.1, P4:U3.3; no longer P4:R2.1, P4:U3.2
- net RX: now also P1:U3.4, P2:U3.4, P3:U3.4, P4:U3.4; no longer P1:U3.3, P2:U3.3, P3:U3.3, P4:U3.3
- net TX: now also P1:U3.2, P2:U3.2, P3:U3.2, P4:U3.2; no longer P1:U3.1, P2:U3.1, P3:U3.1, P4:U3.1
Routing:
- net 3V3_TALON: track 0.00 -> 171.1 mm, vias 0 -> 19
- net 3V3_BULK: track 156.5 -> 0.00 mm, vias 11 -> 0
- net 3V3_TALON+: track 0.00 -> 38.2 mm, vias 0 -> 4
- net GND: track 912.5 -> 944.7 mm, vias 57 -> 59
- net 3V3_AUX_EN: track 55.8 -> 72.0 mm, vias 3 -> 4
- net CSA_EN: track 84.5 -> 90.6 mm
- net 3V3_CORE: track 337.9 -> 343.6 mm, vias 20 -> 21
- net SENSOR_INT: track 86.9 -> 92.3 mm
- net P4:3V3_TALON: track 19.5 -> 14.3 mm, vias 2 -> 0
- net P3:3V3_TALON: track 19.5 -> 14.5 mm, vias 2 -> 0
- net P1:3V3_TALON: track 19.4 -> 14.4 mm, vias 2 -> 0
- net P2:3V3_TALON: track 19.4 -> 14.4 mm, vias 2 -> 0
- net SDA_OB: track 168.2 -> 173.0 mm
- net SCL_OB: track 167.8 -> 172.5 mm
- net 3V3_AUX: track 183.3 -> 178.7 mm
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- added copper zone on layer 1, net 3V3_TALON+
Other:
- board text added: "Particle Status"
- board text added: "Project Kestrel v1.4 Bobby Schulz"
- board text removed: "Project Kestrel v1.3 Bobby Schulz"
