File: Hardware/MainLogger.sch (EAGLE design)
At the start: 202 parts, among them J3 GEMS_POWER_PLUGINPUT_RT, J4 U.FL, J5 SIM_CDNANO_SF72, Q1 DMG3404, Q2 MOSFET_PCH-DMP3036SFG, Q3 MOSFET_PCH-DMP3036SFG, Q4 DMG3404, Q5 NX2301P, Q6 NX2301P, U1 FXMAR2102UMLP, U10 SN74AUP3G34DCU, U11 SIP32431TDFN, U12 LTC4412S6, U13 TCR2LE31ESV, U14 LP59073.3VYKE, U15 MIC22602, U16 BQ25616, U17 TPS61282D, U18 MCP23018QFN, U19 MCP23018QFN, U2 VEML3328, U20 MAX-M8W, U21 MCP79412SOIC, U22 HALL_EFFECT_SI7201, U23 PCA9634QFN, U24 SN74LVC1G17DCK, U25 TPL5010DDC, U26 TPL5010DDC, U27 MB85RC, U28 FXMAR2102UMLP, U29 SIT1552, U3 MMC5633, U4 MXC6655, U5 PAC1934QFN, U6 PAC1934QFN, U7 SHT40, U8 SN74AUP1G08DCK, U9 FXMAR2102UMLP

Commit message: Updated v1.4 for production
Parts:
- added C44, C45: 0.1uF, bschulz_passives:C-EU0.1UFC0402
- added C53, C54: 1uF, bschulz_passives:C-EU1UFC0603
- added R68: 5.6k, bschulz_passives:R-EU_5.6KR0402
- added U30: TCK111G, bschulz:TCK111G
- added U31: FPF2195BUCX, bschulz:FPF2195BUCX
- added U32: (no value), bschulz:SN74LVC1G14DCK
- C23, C29: DIGIKEY (none) -> 490-5523-1-ND; MPN (none) -> GRM21BR61E106KA73L
- C34: value 10uF -> 22uF; device bschulz_passives:C-EU10UFC0805 -> bschulz_passives:C-EU22UFC0805
- L1, L3: DIGIKEY 732-11737-1-ND -> 732-11310-1-ND; MPN 78438357010 -> 78438356010
- R18: device bschulz_passives:R-EU_1KR0603 -> bschulz_passives:R-EU_750R0603
- R27: value 470R -> 220R; device bschulz_passives:R-EU_470R0402 -> bschulz_passives:R-EU_220R0402
- R3: value 0R -> 13.3k; device bschulz_passives:R-EU_0.0R0402 -> bschulz_passives:R-EU_13.3KR0402
- R34, R36: value 10m -> 2m; device bschulz_passives:R-EU_0.01R0805 -> bschulz_passives:R-EU_0.002R0805
- R37: value 10k -> 2.7k; device bschulz_passives:R-EU_10KR0402 -> bschulz_passives:R-EU_2.7KR0402
- R38: device bschulz_passives:R-EU_150KR0603 -> bschulz_passives:R-EU_150KR0402
- R39: device bschulz_passives:R-EU_10KR0603 -> bschulz_passives:R-EU_10KR0402
- R4: value 0R -> 2k; device bschulz_passives:R-EU_0.0R0402 -> bschulz_passives:R-EU_2KR0402
- R43: device bschulz_passives:R-EU_130KR0603 -> bschulz_passives:R-EU_130KR0402
- R44: device bschulz_passives:R-EU_30KR0603 -> bschulz_passives:R-EU_30KR0402
- R50, R51, R52: value 4.7k -> 5.6k; device bschulz_passives:R-EU_4.7KR0603 -> bschulz_passives:R-EU_5.6KR0402
- R56: value 100k -> 130k; device bschulz_passives:R-EU_100KR0402 -> bschulz_passives:R-EU_130KR0402
- R58: value 10k -> 11k; device bschulz_passives:R-EU_10KR0402 -> bschulz_passives:R-EU_11KR0402
- R6, R7: value 2m -> 10m; device bschulz_passives:R-EU_0.002R0805 -> bschulz_passives:R-EU_0.01R0805
- U11: value SIP32431TDFN -> TCK111G; device bschulz:SIP32431TDFN -> bschulz:TCK111G
Connections:
- removed net 3V3_BULK: R7.1, U6.SENSE4-
- new net 3V3_TALON+: C45.1, C54.1, R7.1, U30.VOUT, U31.OUT, U6.SENSE4+
- new net N$19: R68.2, U31.ILIM
- new net N$28: U31.EN, U32G1.Y
- net !FAULT: no longer R1.1
- net 3V3: now also U2.VA, U3.VCC; no longer R1.2
- net 3V3_AUX_EN: now also U30.EN, U32G1.A
- net 3V3_BULK+: now also C53.1, U30.VIN; no longer R7.2, U6.SENSE4+
- net 3V3_CORE: now also C44.1, U31.IN, U32G2.P$V+
- net 3V3_TALON: now also R7.2, U6.SENSE4-; no longer U2.VA, U3.VCC
- net GND: now also C44.2, C45.2, C53.2, C54.2, R68.1, U30.GND, U31.GND, U32G2.P$V-
- net N$1: now also R2.1, U3.1B0; no longer R3.1, U3.2B1
- net N$2: now also R3.1, U3.2B0; no longer R2.1, U3.1B1
- net RX: now also U3.2B1; no longer U3.2B0
- net TX: now also U3.1B1; no longer U3.1B0
